File: kicad/melodyous-micro.kicad_sch (KiCad schematic)
At the start: 11 parts, among them J1 TRS, U1 ProMicro

Commit message: qtpy version
Parts:
- removed JP1: RAW5V, Jumper:SolderJumper-2_P1.3mm_Open_TrianglePad1.0x1.5mm, symbol Jumper:SolderJumper_2_Open
- removed JP2: VCC5V, Jumper:SolderJumper-2_P1.3mm_Open_TrianglePad1.0x1.5mm, symbol Jumper:SolderJumper_2_Open
- removed MCP42010: MCP42010, Package_SO:TSSOP-14-1EP_4.4x5mm_P0.65mm, symbol Potentiometer_Digital:MCP42010
- removed U1: ProMicro, Keebio-Parts:Elite-C-castellated-24pin-holes, symbol keebio:ProMicro
- added U1: qtpy, adafruit:qtpy, symbol MCU_Microchip_SAMD:qtpy
- added U2: MCP41010, Package_SO:SOIC-8_3.9x4.9mm_P1.27mm, symbol Potentiometer_Digital:MCP41010
- POT1: renamed from POTW1; value POT- -> Tape Pot
Connections:
- net +5V: now reaches ISOLATOR1.8 (VCC), R1.2
- net +5V: now also U1.14 (5V), U2.8 (VDD)
- net GND: now reaches ISOLATOR1.5 (GND), R2.2
- net GND: now also U1.13 (GND), U2.4 (VSS)
- net at ISOLATOR1.6 (VO2), R1.1: now also U1.8 (RX)
- new net: U1.11 (MOSI), U2.3 (SI)
- new net: U1.12 (3V3), U2.5 (PA0)
- new net: U1.4 (A3), U2.1 (~{CS})
- new net: U1.9 (SCK), U2.2 (SCK)
- new net: POT1.SPEEDGND, U2.7 (PB0)
- new net: POT1.SPEEDW, U2.6 (PW0)
- no-connect marks 19 -> 7
Other:
- moved on the sheet: POT1
